File: rear_distribution.kicad_pcb (KiCad board)
At the start: 4 copper layers, 126 parts, among them J1 Conn_01x08, J11 Conn_01x35, J2 Conn_01x06, J21 Conn_01x23, J3 10067847-001RLF, J31 Conn_01x23, J41 Conn_01x23, J51 Conn_01x08, J61 Conn_01x08, J71 Conn_01x02, J81 Conn_01x02, J82 Conn_01x02, J83 Conn_01x04, J84 Conn_01x04, J85 Conn_01x02, J91 Conn_01x02, J92 Conn_01x02, J93 Conn_01x04, J94 Conn_01x03, J95 Conn_01x08, K1 G2RL-1A, Q1 DMN6075S, Q2 DMN6075S, SW1 SW_Push, U1 TPS7B88, U2 MCP1700x-330xxMB, U3 STM32F103C8Tx, U4 SN65HVD1050D, U5 TCA9535PWR, Y1 8M, Y2 32.768k

Commit message: pcb: Add layout progress so far
Parts:
- removed the J71 at (-145.0, 174.7)
- removed the J84 at (-102.8, 206.4)
- removed R11, R12: 10k, Resistor_SMD:R_0603_1608Metric
- J1: value Conn_01x08 -> Conn_01x06; footprint yfs:MolexMicrofitPlus1x8 -> yfs:MolexMicrofitPlus2x3
- moved BT1 491.7 mm to (213.0, 111.0)
- moved U4 471.0 mm to (178.5, 121.5), turned to -90 degrees
- moved Y1 467.4 mm to (175.5, 106.0), turned to 90 degrees
- moved J84 446.5 mm to (241.0, 98.0), turned to 90 degrees
- moved JP61 441.8 mm to (233.0, 67.0), turned to 90 degrees
- moved C8 438.7 mm to (179.0, 101.5)
- moved U3 430.6 mm to (166.0, 106.0), turned to 180 degrees
- moved RN5 430.5 mm to (186.0, 104.0), turned to 180 degrees
- moved C13 429.5 mm to (180.0, 110.5)
- moved C11 429.4 mm to (179.5, 104.5)
- moved RN6 429.1 mm to (186.0, 97.0)
- moved J85 428.4 mm to (241.0, 110.0), turned to 90 degrees
- moved C15 427.8 mm to (178.5, 116.5)
- moved C9 427.7 mm to (170.5, 112.0), turned to -90 degrees
- moved C12 427.5 mm to (180.0, 113.5)
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- renumbered F81 to F71, F91 to F81, J81 to J71, J82 to J72, J83 to J73, J85 to J74, J91 to J81, J92 to J82, J93 to J83, J94 to J84, J95 to J85
Connections:
- net Net-(D1-A2) renamed /Microcontroller/12V_FUSED
- net Net-(D3-K) renamed /Microcontroller/12V_SAFE
- F13 pad 1: Net-(F13-Pad1) -> +12V
- F13 pad 2: +12V -> 12V_COOLANT_IN
- J1 pad 2: GND -> +5V
- J1 pad 3: GND -> /Microcontroller/RADIO_TX
- J1 pad 4: /Microcontroller/RADIO_CTS -> /Microcontroller/RADIO_RTS
- J1 pad 5: /Microcontroller/RADIO_RTS -> /Microcontroller/RADIO_CTS
- J11 pad 1: GND -> SDN_RIGHT_ESTOP_OUT
- J11 pad 10: unconnected-(J11-Pin_10-Pad10) -> 12V_TSAL_LED
- J11 pad 11: SDN_BSPD_OUT -> 12V_BRAKE_LIGHT
- J11 pad 12: IMD_RESET -> 12V_COOLANT
- J11 pad 13: BMS_RESET -> SDN_LEFT_ESTOP_IN
- J11 pad 2: GND -> SDN_BSPD_OUT
- J11 pad 20: BRAKE_SWITCH_OUT -> TSAL_GREEN
- J11 pad 24: TSAL_GREEN -> unconnected-(J11-Pin_24-Pad24)
- J11 pad 25: 12V_TSAL_LED -> unconnected-(J11-Pin_25-Pad25)
- J11 pad 26: GND_BRAKE_LIGHT -> unconnected-(J11-Pin_26-Pad26)
- J11 pad 27: 12V_BRAKE_LIGHT -> unconnected-(J11-Pin_27-Pad27)
- J11 pad 29: 12V_COOLANT -> unconnected-(J11-Pin_29-Pad29)
- J11 pad 3: GND -> SDN_RIGHT_ESTOP_IN
- J11 pad 30: SDN_TSMS_OUT -> unconnected-(J11-Pin_30-Pad30)
- J11 pad 31: SDN_TSMS_IN -> unconnected-(J11-Pin_31-Pad31)
- J11 pad 32: SDN_RIGHT_ESTOP_OUT -> unconnected-(J11-Pin_32-Pad32)
- J11 pad 33: SDN_RIGHT_ESTOP_IN -> unconnected-(J11-Pin_33-Pad33)
- J11 pad 34: SDN_LEFT_ESTOP_OUT -> unconnected-(J11-Pin_34-Pad34)
- J11 pad 35: SDN_LEFT_ESTOP_IN -> unconnected-(J11-Pin_35-Pad35)
- J11 pad 4: GND -> SDN_LEFT_ESTOP_OUT
- J11 pad 5: unconnected-(J11-Pin_5-Pad5) -> SDN_TSMS_IN
- J11 pad 6: unconnected-(J11-Pin_6-Pad6) -> SDN_TSMS_OUT
- J11 pad 8: unconnected-(J11-Pin_8-Pad8) -> GND_BRAKE_LIGHT
- J11 pad 9: unconnected-(J11-Pin_9-Pad9) -> BRAKE_SWITCH_OUT
- J31 pad 1: 12V_PRCHG -> 12V_FAN
- J31 pad 10: BMS_OK -> IMD_OK
- J31 pad 11: IMD_OK -> IMD_PWM
- J31 pad 12: IMD_PWM -> DISCHG
- J31 pad 13: DISCHG -> CANL
- J31 pad 14: PRCHG_INT -> CANH
- J31 pad 15: PRCHG_ACT -> AIR-_ACT
- J31 pad 16: AIR-_INT -> SDN_TSAC_IN
- J31 pad 17: AIR-_ACT -> 12V_PRCHG
- J31 pad 18: AIR+_INT -> GND
- J31 pad 19: AIR+_ACT -> GND
- J31 pad 20: HV_DET -> GND
- J31 pad 21: GND -> AIR-_INT
- J31 pad 22: GND -> PRCHG_ACT
- J31 pad 23: GND -> PRCHG_INT
- J31 pad 3: 12V_HV_DET -> 12V_BMS
- J31 pad 4: 12V_FAN -> 12V_HV_DET
- J31 pad 5: 12V_BMS -> HV_DET
- J31 pad 7: CANH -> AIR+_ACT
- J31 pad 8: CANL -> AIR+_INT
- J31 pad 9: SDN_TSAC_IN -> BMS_OK
- J41 pad 19: DTI_OUT_1 -> unconnected-(J41-Pin_19-Pad19)
- J41 pad 20: DTI_OUT_2 -> unconnected-(J41-Pin_20-Pad20)
- J41 pad 21: DTI_IN_1 -> unconnected-(J41-Pin_21-Pad21)
- J41 pad 22: DTI_IN_2 -> unconnected-(J41-Pin_22-Pad22)
- J61 pad 4: SDN_AUX_IN -> SDN_AUX_OUT
- J61 pad 5: SDN_AUX_OUT -> SDN_AUX_IN
- K1 pad 13: 12V_COOLANT -> 12V_COOLANT_IN
- K1 pad 14: Net-(F13-Pad1) -> 12V_COOLANT
- RN1 pad 1: 12V_AUX -> 12V_COOLANT_IN
- RN1 pad 2: 12V_BMS -> 12V_BRAKE_LIGHT
- RN1 pad 3: 12V_COOLANT -> 12V_TSAL_LED
- RN1 pad 6: /12V_COOLANT_SAMPLE -> /12V_TSAL_LED_SAMPLE
- RN1 pad 7: /12V_BMS_SAMPLE -> /12V_BRAKE_LIGHT_SAMPLE
- RN1 pad 8: /12V_AUX_SAMPLE -> /12V_COOLANT_SAMPLE
- RN10 pad 1: /SDN_RIGHT_ESTOP_SAMPLE -> /SDN_AUX_SAMPLE
- RN10 pad 2: /SDN_HVD_SAMPLE -> /SDN_FRONT_SAMPLE
- RN10 pad 3: /SDN_AUX_SAMPLE -> /SDN_LATCH_SAMPLE
- RN10 pad 4: /SDN_TSMS_SAMPLE -> /SDN_LEFT_ESTOP_SAMPLE
- RN11 pad 1: BMS_OK -> SDN_BSPD_OUT
- RN11 pad 2: IMD_OK -> SDN_LEFT_ESTOP_OUT
- RN11 pad 3: DTI_OK -> SDN_TSMS_OUT
- RN11 pad 4: DISCHG -> SDN_AUX_OUT
- RN11 pad 5: /DISCHG_OK_SAMPLE -> /SDN_TSMS_SAMPLE
- RN11 pad 6: /DTI_OK_SAMPLE -> /SDN_BSPD_SAMPLE
- RN11 pad 7: /IMD_OK_SAMPLE -> /SDN_RIGHT_ESTOP_SAMPLE
- RN11 pad 8: /BMS_OK_SAMPLE -> /SDN_HVD_SAMPLE
- RN12 pad 1: /BMS_OK_SAMPLE -> /SDN_HVD_SAMPLE
- RN12 pad 2: /IMD_OK_SAMPLE -> /SDN_RIGHT_ESTOP_SAMPLE
- RN12 pad 3: /DTI_OK_SAMPLE -> /SDN_BSPD_SAMPLE
- RN12 pad 4: /DISCHG_OK_SAMPLE -> /SDN_TSMS_SAMPLE
- RN2 pad 1: /12V_AUX_SAMPLE -> /12V_COOLANT_SAMPLE
- RN2 pad 2: /12V_BMS_SAMPLE -> /12V_BRAKE_LIGHT_SAMPLE
- RN2 pad 3: /12V_COOLANT_SAMPLE -> /12V_TSAL_LED_SAMPLE
- RN3 pad 1: 12V_ENERGY_METER -> 12V_LATCH
- RN3 pad 2: 12V_FAN -> 12V_ENERGY_METER
- RN3 pad 3: 12V_IMD -> DTI_OK
- RN3 pad 4: 12V_PRCHG -> BRAKE_SWITCH_OUT
- RN3 pad 5: /12V_PRCHG_SAMPLE -> /BRAKE_SWITCH_SAMPLE
- RN3 pad 6: /12V_IMD_SAMPLE -> /DTI_OK_SAMPLE
- RN3 pad 7: /12V_FAN_SAMPLE -> /12V_ENERGY_METER_SAMPLE
- RN3 pad 8: /12V_ENERGY_METER_SAMPLE -> /12V_LATCH_SAMPLE
- RN4 pad 1: /12V_ENERGY_METER_SAMPLE -> /12V_LATCH_SAMPLE
- RN4 pad 2: /12V_FAN_SAMPLE -> /12V_ENERGY_METER_SAMPLE
- RN4 pad 3: /12V_IMD_SAMPLE -> /DTI_OK_SAMPLE
- RN4 pad 4: /12V_PRCHG_SAMPLE -> /BRAKE_SWITCH_SAMPLE
- RN5 pad 1: 12V_LATCH -> 12V_PRCHG
- RN5 pad 2: 12V_TSAL_LED -> 12V_FAN
- RN5 pad 3: BRAKE_SWITCH_OUT -> 12V_IMD
- RN5 pad 4: IMD_PWM -> 12V_BMS
- RN5 pad 5: /IMD_PWM_SAMPLE -> /12V_BMS_SAMPLE
- RN5 pad 6: /BRAKE_SWITCH_SAMPLE -> /12V_IMD_SAMPLE
- RN5 pad 7: /12V_TSAL_LED_SAMPLE -> /12V_FAN_SAMPLE
- RN5 pad 8: /12V_LATCH_SAMPLE -> /12V_PRCHG_SAMPLE
- RN6 pad 1: /12V_LATCH_SAMPLE -> /12V_PRCHG_SAMPLE
- RN6 pad 2: /12V_TSAL_LED_SAMPLE -> /12V_FAN_SAMPLE
- RN6 pad 3: /BRAKE_SWITCH_SAMPLE -> /12V_IMD_SAMPLE
- RN6 pad 4: /IMD_PWM_SAMPLE -> /12V_BMS_SAMPLE
- RN7 pad 1: SDN_BSPD_OUT -> IMD_PWM
- RN7 pad 2: SDN_FRONT_OUT -> IMD_OK
- RN7 pad 3: SDN_LATCH_OUT -> BMS_OK
- RN7 pad 4: SDN_LEFT_ESTOP_OUT -> DISCHG
- RN7 pad 5: /SDN_LEFT_ESTOP_SAMPLE -> /DISCHG_SAMPLE
- RN7 pad 6: /SDN_LATCH_SAMPLE -> /BMS_OK_SAMPLE
- RN7 pad 7: /SDN_FRONT_SAMPLE -> /IMD_OK_SAMPLE
- RN7 pad 8: /SDN_BSPD_SAMPLE -> /IMD_PWM_SAMPLE
- RN8 pad 1: /SDN_BSPD_SAMPLE -> /IMD_PWM_SAMPLE
- RN8 pad 2: /SDN_FRONT_SAMPLE -> /IMD_OK_SAMPLE
- RN8 pad 3: /SDN_LATCH_SAMPLE -> /BMS_OK_SAMPLE
- RN8 pad 4: /SDN_LEFT_ESTOP_SAMPLE -> /DISCHG_SAMPLE
- RN9 pad 1: SDN_RIGHT_ESTOP_OUT -> SDN_FRONT_OUT
- RN9 pad 3: SDN_AUX_OUT -> SDN_RIGHT_ESTOP_OUT
- RN9 pad 4: SDN_TSMS_OUT -> SDN_LATCH_OUT
- RN9 pad 5: /SDN_TSMS_SAMPLE -> /SDN_LEFT_ESTOP_SAMPLE
- RN9 pad 6: /SDN_AUX_SAMPLE -> /SDN_LATCH_SAMPLE
- RN9 pad 7: /SDN_HVD_SAMPLE -> /SDN_FRONT_SAMPLE
- RN9 pad 8: /SDN_RIGHT_ESTOP_SAMPLE -> /SDN_AUX_SAMPLE
- U3 pad 10: /12V_AUX_SAMPLE -> /12V_BMS_SAMPLE
- U3 pad 11: /12V_BMS_SAMPLE -> /12V_IMD_SAMPLE
- U3 pad 12: /12V_COOLANT_SAMPLE -> /12V_FAN_SAMPLE
- U3 pad 13: /12V_DTI_SAMPLE -> /12V_PRCHG_SAMPLE
- U3 pad 14: /12V_ENERGY_METER_SAMPLE -> /12V_COOLANT_SAMPLE
- U3 pad 15: /12V_FAN_SAMPLE -> /12V_BRAKE_LIGHT_SAMPLE
- U3 pad 16: /12V_IMD_SAMPLE -> /12V_TSAL_LED_SAMPLE
- U3 pad 17: /12V_PRCHG_SAMPLE -> /12V_DTI_SAMPLE
- U3 pad 19: /12V_TSAL_LED_SAMPLE -> /12V_ENERGY_METER_SAMPLE
- U3 pad 20: MCU_COOLANT -> /DTI_OK_SAMPLE
- U3 pad 21: /IMD_PWM_SAMPLE -> /BRAKE_SWITCH_SAMPLE
- U3 pad 22: SD_DETECT -> unconnected-(U3-PB11-Pad22)
- U3 pad 29: MCU_BRAKE -> SD_DETECT
- U3 pad 41: /BRAKE_SWITCH_SAMPLE -> /IMD_PWM_SAMPLE
- U5 pad 10: /SDN_AUX_SAMPLE -> /SDN_RIGHT_ESTOP_SAMPLE
- U5 pad 11: /SDN_TSMS_SAMPLE -> /SDN_HVD_SAMPLE
- U5 pad 13: /BMS_OK_SAMPLE -> MCU_COOLANT
- U5 pad 14: /IMD_OK_SAMPLE -> /DISCHG_SAMPLE
- U5 pad 15: /DTI_OK_SAMPLE -> /BMS_OK_SAMPLE
- U5 pad 16: /DISCHG_OK_SAMPLE -> /IMD_OK_SAMPLE
- U5 pad 17: DTI_OUT_1 -> MCU_BRAKE
- U5 pad 18: DTI_OUT_2 -> unconnected-(U5-P15-Pad18)
- U5 pad 19: DTI_IN_1 -> unconnected-(U5-P16-Pad19)
- U5 pad 20: DTI_IN_2 -> unconnected-(U5-P17-Pad20)
- U5 pad 4: /SDN_BSPD_SAMPLE -> /SDN_LEFT_ESTOP_SAMPLE
- U5 pad 5: /SDN_FRONT_SAMPLE -> /SDN_LATCH_SAMPLE
- U5 pad 6: /SDN_LATCH_SAMPLE -> /SDN_FRONT_SAMPLE
- U5 pad 7: /SDN_LEFT_ESTOP_SAMPLE -> /SDN_AUX_SAMPLE
- U5 pad 8: /SDN_RIGHT_ESTOP_SAMPLE -> /SDN_TSMS_SAMPLE
- U5 pad 9: /SDN_HVD_SAMPLE -> /SDN_BSPD_SAMPLE
Routing:
- net CANH: track 0.00 -> 261.4 mm, vias 0 -> 2
- net CANL: track 0.00 -> 255.6 mm, vias 0 -> 2
- net SDN_AUX_OUT: track 0.00 -> 249.0 mm
- net SDN_FRONT_IN: track 0.00 -> 225.3 mm
- net SDN_LATCH_OUT: track 0.00 -> 181.5 mm
- net DISCHG: track 0.00 -> 181.1 mm, vias 0 -> 1
- net 12V_ENERGY_METER: track 0.00 -> 125.3 mm
- net /Microcontroller/RADIO_TX: track 0.00 -> 117.4 mm, vias 0 -> 2
- net /Microcontroller/RADIO_RTS: track 0.00 -> 113.7 mm, vias 0 -> 2
- net /Microcontroller/RADIO_CTS: track 0.00 -> 113.0 mm, vias 0 -> 2
- net /Microcontroller/RADIO_RX: track 0.00 -> 112.4 mm, vias 0 -> 2
- net +5V: track 0.00 -> 95.4 mm
- net SDN_HVD_OUT: track 0.00 -> 78.6 mm
- net 12V_HV_DET: track 0.00 -> 78.6 mm
- net 12V_BRAKE_LIGHT: track 0.00 -> 70.2 mm
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- added copper zone on F.Cu, net +12V
- added copper zone on In1.Cu, net +12V
- added copper zone on F.Cu, net +5V
- added copper zone on F.Cu, net /Microcontroller/12V_FUSED
- added copper zone on F.Cu, net /Microcontroller/12V_SAFE
- added copper zone on B.Cu, net GND
- added copper zone on F.Cu, net GND
- added copper zone on In2.Cu, net GND
Other:
- board outline added: 210 x 100 mm

Commit message: *: Tentatively finish everything
Parts:
- removed NT1: NetTie_3_Tee, NetTie:NetTie-3_SMD_Pad0.5mm
- removed TP3, TP4: TestPoint, TestPoint:TestPoint_Keystone_5000-5004_Miniature
- added G***: LOGO, LOGO, B.Cu at (220.5, 110.9)
- added kibuzzard-6940937D: G***, kibuzzard-6940937D, F.Cu at (233.8, 108.7)
- added kibuzzard-6A356FF1: G***, kibuzzard-6A356FF1, F.Cu at (53.5, 87.8)
- added kibuzzard-6A357015: G***, kibuzzard-6A357015, F.Cu at (54.5, 78.8)
- added kibuzzard-6A357015: G***, kibuzzard-6A357015, F.Cu at (54.5, 69.8)
- added kibuzzard-6A35710C: G***, kibuzzard-6A35710C, F.Cu at (55.0, 120.7)
- added kibuzzard-6A3571FC: G***, kibuzzard-6A3571FC, F.Cu at (60.4, 109.1)
- added kibuzzard-6A3572FA: G***, kibuzzard-6A3572FA, F.Cu at (235.0, 72.7)
- added kibuzzard-6A3574B6: G***, kibuzzard-6A3574B6, F.Cu at (233.8, 96.7)
- added kibuzzard-6A35750C: G***, kibuzzard-6A35750C, F.Cu at (235.0, 87.8)
- added kibuzzard-6A357544: G***, kibuzzard-6A357544, F.Cu at (235.0, 63.8)
- J3: value 10067847-001RLF -> 47219-2001; footprint yfs:10067847-001RLF_AMP -> yfs:Molex_SD_Slot_47219-2001
- NT8: moved to B.Cu
- moved TP6 273.7 mm to (202.6, 96.0)
- moved TP1 219.9 mm to (117.5, 112.0)
- moved C19 188.9 mm to (81.5, 98.5)
- moved R10 184.5 mm to (81.5, 101.5), turned to 180 degrees
- moved NT8 170.5 mm to (249.0, 123.0), turned to 90 degrees
- moved R7 168.3 mm to (61.0, 104.0)
- moved R5 166.2 mm to (61.0, 100.0)
- moved R6 166.1 mm to (61.0, 102.0)
- moved R8 164.8 mm to (61.0, 96.0)
- moved R9 164.6 mm to (61.0, 98.0)
- moved TP2 154.1 mm to (53.5, 100.0)
- moved J3 123.9 mm to (71.0, 100.0)
- moved JP61 12.5 mm to (236.5, 55.0), turned to 180 degrees
- moved NT2 3.20 mm to (149.0, 141.0), turned to 0 degrees
- moved J1 0.25 mm to (49.2, 116.0)
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Connections:
- J11 pad 14: +12V -> unconnected-(J11-Pin_14-Pad14)
- J11 pad 15: +12V -> unconnected-(J11-Pin_15-Pad15)
- J11 pad 16: +12V -> unconnected-(J11-Pin_16-Pad16)
- J11 pad 17: unconnected-(J11-Pin_17-Pad17) -> +12V
- J11 pad 18: unconnected-(J11-Pin_18-Pad18) -> +12V
- J11 pad 19: unconnected-(J11-Pin_19-Pad19) -> +12V
- J11 pad 20: TSAL_GREEN -> +12V
- J11 pad 21: BRAKE_SWITCH_IN -> +12V
- J11 pad 22: GND_TSAL_LED -> BRAKE_SWITCH_IN
- J11 pad 28: GND_COOLANT -> unconnected-(J11-Pin_28-Pad28)
- J11 pad 29: unconnected-(J11-Pin_29-Pad29) -> GND
- J11 pad 30: unconnected-(J11-Pin_30-Pad30) -> GND
- J11 pad 31: unconnected-(J11-Pin_31-Pad31) -> GND
- J11 pad 32: unconnected-(J11-Pin_32-Pad32) -> GND
- J11 pad 33: unconnected-(J11-Pin_33-Pad33) -> GND
- J11 pad 34: unconnected-(J11-Pin_34-Pad34) -> GND
- J11 pad 35: unconnected-(J11-Pin_35-Pad35) -> TSAL_GREEN
- J3 pad 1: SD_CS -> /Microcontroller/SD_DAT2
- J3 pad 2: SD_MOSI -> SD_CS
- J3 pad 3: GND -> SD_MOSI
- J73 pad 2: DTI_OK -> BMS_OK
- J73 pad 4: BMS_OK -> DTI_OK
- RN7 pad 1: IMD_PWM -> BMS_OK
- RN7 pad 3: BMS_OK -> IMD_PWM
- RN7 pad 6: /BMS_OK_SAMPLE -> /IMD_PWM_SAMPLE
- RN7 pad 8: /IMD_PWM_SAMPLE -> /BMS_OK_SAMPLE
- RN8 pad 1: /IMD_PWM_SAMPLE -> /BMS_OK_SAMPLE
- RN8 pad 3: /BMS_OK_SAMPLE -> /IMD_PWM_SAMPLE
- U3 pad 29: SD_DETECT -> unconnected-(U3-PA8-Pad29)
Routing:
- net TSAL_GREEN: track 0.00 -> 300.7 mm, vias 0 -> 1
- net +3V3: track 10.6 -> 218.3 mm, vias 0 -> 7
- net SDN_HVD_OUT: track 78.6 -> 282.8 mm
- net DTI_OK: track 0.00 -> 158.6 mm, vias 0 -> 4
- net BMS_OK: track 19.0 -> 159.9 mm
- net IMD_OK: track 23.6 -> 164.4 mm
- net SD_MOSI: track 0.00 -> 114.1 mm, vias 0 -> 2
- net TSAL_RED: track 0.00 -> 111.7 mm
- net SD_MISO: track 0.00 -> 109.8 mm, vias 0 -> 2
- net SD_CS: track 0.00 -> 109.8 mm, vias 0 -> 2
- net SD_SCK: track 0.00 -> 102.7 mm, vias 0 -> 2
- net 12V_LATCH: track 18.8 -> 110.0 mm
- net +5V: track 95.4 -> 178.2 mm, vias 0 -> 4
- net SDN_FRONT_OUT: track 36.1 -> 118.5 mm, vias 0 -> 2
- net SDN_AUX_IN: track 27.6 -> 108.2 mm, vias 0 -> 1
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- added copper zone on F.Cu, net +3V3
Other:
- board text added: "${PCB_DATE}"
- board text added: "+5V"
- board text added: "+5VL"
- board text added: "12V_UPS"
- board text added: "3V3"
- board text added: "5V"
- board text added: "AIR+_ACT"
- board text added: "AIR+_INT"
- board text added: "AIR-_ACT"
- board text added: "AIR-_INT"
- board text added: "BMS"
- board text added: "BMS_OK"
- board text added: "BY OWEN S"
- board text added: "CTS"
- board text added: "DET"
- board text added: "DTI_OK"
- board text added: "GND"
- board text added: "GREEN"
- board text added: "IMD"
- board text added: "IMD_OK"
- board text added: "IN"
- board text added: "LV+"
- board text added: "LV-"
- board text added: "OUT"
- board text added: "Owen Smith"
- board text added: "PREC_ACT"
- board text added: "PREC_INT"
- board text added: "REAR DISTRIBUTION"
- board text added: "RED"
- board text added: "REV ${REVISION}"
- board text added: "RTS"
- board text added: "RX"
- board text added: "TX"
- board text added: "york-fs/rear-distribution"
