File: rear_distribution.kicad_pcb (KiCad board)
At the start: 4 copper layers, 210 x 100 mm, 134 parts, among them J1 Conn_01x06, J11 Conn_01x35, J2 Conn_01x06, J21 Conn_01x23, J3 47219-2001, J31 Conn_01x23, J41 Conn_01x23, J51 Conn_01x08, J61 Conn_01x08, J71 Conn_01x02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

Commit message: schematic: Cleanup BOM
Parts:
- renumbered CANH to TP4, CANL to TP5
Other:
- board text added: "CANH"
- board text added: "CANL"
