File: rear_distribution.kicad_pcb (KiCad board)
At the start: 4 copper layers, 210 x 100 mm, 134 parts, among them J1 Conn_01x06, J11 Conn_01x35, J2 Conn_01x06, J21 Conn_01x23, J3 47219-2001, J31 Conn_01x23, J41 Conn_01x23, J51 Conn_01x08, J61 Conn_01x08, J71 Conn_01x02, J72 Conn_01x02, J73 Conn_01x04, J74 Conn_01x02, J81 Conn_01x02, J82 Conn_01x02, J83 Conn_01x04, J84 Conn_01x03, J85 Conn_01x08, K1 G2RL-1A, Q1 DMN6075S, Q2 DMN6075S, SW1 SW_Push, U1 TPS7B88, U2 MCP1700x-330xxMB, U3 STM32F103C8Tx, U4 SN65HVD1050D, U5 TCA9535PWR, Y1 8M, Y2 32.768k

Commit message: schematic: Rename some nets to match naming scheme
Connections:
- net BMS_INDICATOR_GND renamed GND_BMS_INDICATOR
- net IMD_INDICATOR_GND renamed GND_IMD_INDICATOR
Changed lines of the file:
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@@
 	(net 57 "TSAL_RED")
 	(net 58 "BRAKE_SWITCH_IN")
-	(net 59 "IMD_INDICATOR_GND")
-	(net 60 "BMS_INDICATOR_GND")
+	(net 59 "GND_IMD_INDICATOR")
+	(net 60 "GND_BMS_INDICATOR")
 	(net 61 "SDN_FRONT_OUT")
 	(net 62 "DISCHG")
@@
 			(layers "*.Cu" "*.Mask")
 			(remove_unused_layers no)
-			(net 59 "IMD_INDICATOR_GND")
+			(net 59 "GND_IMD_INDICATOR")
 			(pinfunction "Pin_1")
 			(pintype "passive")
@@
 			(layers "*.Cu" "*.Mask")
 			(remove_unused_layers no)
-			(net 60 "BMS_INDICATOR_GND")
+			(net 60 "GND_BMS_INDICATOR")
 			(pinfunction "Pin_2")
 			(pintype "passive")
@@
 			(layers "*.Cu" "*.Mask")
 			(remove_unused_layers no)
-			(net 59 "IMD_INDICATOR_GND")
+			(net 59 "GND_IMD_INDICATOR")
 			(pinfunction "Pin_3")
 			(pintype "passive")
@@
 			(layers "*.Cu" "*.Mask")
 			(remove_unused_layers no)
-			(net 60 "BMS_INDICATOR_GND")
+			(net 60 "GND_BMS_INDICATOR")
 			(pinfunction "Pin_9")
 			(pintype "passive")
