File: microcontroller.kicad_sch (KiCad schematic)
At the start: 52 parts, among them J1 Conn_01x06, J2 Conn_01x06, J3 47219-2001, SW1 SW_Push, U1 TPS7B88, U2 MCP1700x-330xxMB, U3 STM32F103C8Tx, U4 SN65HVD1050D, U5 TCA9535PWR, Y1 8M, Y2 32.768k

Commit message: schematic: Exclude some test points from the BOM
Parts:
- TP2, TP3, TP4, TP5: now left out of the parts list
Changed lines of the file:
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@@
 		(unit 1)
 		(exclude_from_sim no)
-		(in_bom yes)
+		(in_bom no)
 		(on_board yes)
 		(dnp no)
@@
 		(unit 1)
 		(exclude_from_sim no)
-		(in_bom yes)
+		(in_bom no)
 		(on_board yes)
 		(dnp no)
@@
 		(unit 1)
 		(exclude_from_sim no)
-		(in_bom yes)
+		(in_bom no)
 		(on_board yes)
 		(dnp no)
@@
 		(unit 1)
 		(exclude_from_sim no)
-		(in_bom yes)
+		(in_bom no)
 		(on_board yes)
 		(dnp no)

Commit message: *: Fix shutdown labelling mismatch
Connections:
- net SDN_AUX_SAMPLE: now also U5.8 (P04); no longer U5.7 (P03)
- net SDN_BSPD_SAMPLE: now also U5.11 (P07); no longer U5.9 (P05)
- net SDN_FRONT_SAMPLE: now also U5.7 (P03); no longer U5.6 (P02)
- net SDN_HVD_SAMPLE: now also U5.6 (P02); no longer U5.11 (P07)
- net SDN_LATCH_SAMPLE: now also U5.4 (P00); no longer U5.5 (P01)
- net SDN_LEFT_ESTOP_SAMPLE: now also U5.10 (P06); no longer U5.4 (P00)
- net SDN_RIGHT_ESTOP_SAMPLE: now also U5.5 (P01); no longer U5.10 (P06)
- net SDN_TSMS_SAMPLE: now also U5.9 (P05); no longer U5.8 (P04)
Changed lines of the file:
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@@
+		)
+	)
+	(hierarchical_label "12V_LATCH_SAMPLE"
+		(shape input)
+		(at 105.41 133.35 0)
+		(effects
+			(font
+				(size 1 1)
+			)
+			(justify left)
+		)
+	)
+	(hierarchical_label "BRAKE_SWITCH_SAMPLE"
+		(shape input)
+		(at 67.31 158.75 180)
+		(effects
+			(font
+				(size 1 1)
+			)
+			(justify right)
 		)
 	)
 	(hierarchical_label "SDN_BSPD_SAMPLE"
 		(shape input)
+		(at 142.24 55.88 180)
+		(effects
+			(font
+				(size 1 1)
+			)
+			(justify right)
+		)
+	)
+	(hierarchical_label "SDN_AUX_SAMPLE"
+		(shape input)
+		(at 142.24 48.26 180)
+		(effects
+			(font
+				(size 1 1)
+			)
+			(justify right)
+		)
+	)
+	(hierarchical_label "DTI_OK_SAMPLE"
+		(shape input)
+		(at 67.31 151.13 180)
+		(effects
+			(font
+				(size 1 1)
+			)
+			(justify right)
+		)
+	)
+	(hierarchical_label "12V_TSAL_LED_SAMPLE"
+		(shape input)
+		(at 105.41 128.27 0)
+		(effects
+			(font
+				(size 1 1)
+			)
+			(justify left)
+		)
+	)
+	(hierarchical_label "BMS_OK_SAMPLE"
+		(shape input)
+		(at 142.24 66.04 180)
+		(effects
+			(font
+				(size 1 1)
+			)
+			(justify right)
+		)
+	)
+	(hierarchical_label "12V_COOLANT_SAMPLE"
+		(shape input)
+		(at 105.41 123.19 0)
+		(effects
+			(font
+				(size 1 1)
+			)
+			(justify left)
+		)
+	)
+	(hierarchical_label "12V_BRAKE_LIGHT_SAMPLE"
+		(shape input)
+		(at 105.41 125.73 0)
+		(effects
+			(font
+				(size 1 1)
+			)
+			(justify left)
+		)
+	)
+	(hierarchical_label "DISCHG_SAMPLE"
+		(shape input)
+		(at 142.24 63.5 180)
+		(effects
+			(font
+				(size 1 1)
+			)
+			(justify right)
+		)
+	)
+	(hierarchical_label "IMD_PWM_SAMPLE"
+		(shape input)
+		(at 67.31 156.21 180)
+		(effects
+			(font
+				(size 1 1)
+			)
+			(justify right)
+		)
+	)
+	(hierarchical_label "SDN_LEFT_ESTOP_SAMPLE"
+		(shape input)
+		(at 142.24 53.34 180)
+		(effects
+			(font
+				(size 1 1)
+			)
+			(justify right)
+		)
+	)
+	(hierarchical_label "SDN_FRONT_SAMPLE"
+		(shape input)
+		(at 142.24 45.72 180)
+		(effects
+			(font
+				(size 1 1)
+			)
+			(justify right)
+		)
+	)
+	(hierarchical_label "12V_DTI_SAMPLE"
+		(shape input)
+		(at 105.41 130.81 0)
+		(effects
+			(font
+				(size 1 1)
+			)
+			(justify left)
+		)
+	)
+	(hierarchical_label "12V_ENERGY_METER_SAMPLE"
+		(shape input)
+		(at 105.41 135.89 0)
+		(effects
+			(font
+				(size 1 1)
+			)
+			(justify left)
+		)
+	)
+	(hierarchical_label "SDN_TSMS_SAMPLE"
+		(shape input)
 		(at 142.24 50.8 180)
 		(effects
@@
 		)
 	)
-	(hierarchical_label "12V_LATCH_SAMPLE"
-		(shape input)
-		(at 105.41 133.35 0)
-		(effects
-			(font
-				(size 1 1)
-			)
-			(justify left)
-		)
-	)
-	(hierarchical_label "BRAKE_SWITCH_SAMPLE"
-		(shape input)
-		(at 67.31 158.75 180)
-		(effects
-			(font
-				(size 1 1)
-			)
-			(justify right)
-		)
-	)
-	(hierarchical_label "DTI_OK_SAMPLE"
-		(shape input)
-		(at 67.31 151.13 180)
-		(effects
-			(font
-				(size 1 1)
-			)
-			(justify right)
-		)
-	)
-	(hierarchical_label "SDN_AUX_SAMPLE"
-		(shape input)
-		(at 142.24 45.72 180)
-		(effects
-			(font
-				(size 1 1)
-			)
-			(justify right)
-		)
-	)
-	(hierarchical_label "12V_TSAL_LED_SAMPLE"
-		(shape input)
-		(at 105.41 128.27 0)
-		(effects
-			(font
-				(size 1 1)
-			)
-			(justify left)
-		)
-	)
-	(hierarchical_label "SDN_LEFT_ESTOP_SAMPLE"
+	(hierarchical_label "12V_FAN_SAMPLE"
+		(shape input)
+		(at 105.41 118.11 0)
+		(effects
+			(font
+				(size 1 1)
+			)
+			(justify left)
+		)
+	)
+	(hierarchical_label "SDN_HVD_SAMPLE"
+		(shape input)
+		(at 142.24 43.18 180)
+		(effects
+			(font
+				(size 1 1)
+			)
+			(justify right)
+		)
+	)
+	(hierarchical_label "12V_IMD_SAMPLE"
+		(shape input)
+		(at 105.41 115.57 0)
+		(effects
+			(font
+				(size 1 1)
+			)
+			(justify left)
+		)
+	)
+	(hierarchical_label "12V_BMS_SAMPLE"
+		(shape input)
+		(at 105.41 113.03 0)
+		(effects
+			(font
+				(size 1 1)
+			)
+			(justify left)
+		)
+	)
+	(hierarchical_label "IMD_OK_SAMPLE"
+		(shape input)
+		(at 142.24 68.58 180)
+		(effects
+			(font
+				(size 1 1)
+			)
+			(justify right)
+		)
+	)
+	(hierarchical_label "SDN_RIGHT_ESTOP_SAMPLE"
+		(shape input)
+		(at 142.24 40.64 180)
+		(effects
+			(font
+				(size 1 1)
+			)
+			(justify right)
+		)
+	)
+	(hierarchical_label "SDN_LATCH_SAMPLE"
 		(shape input)
 		(at 142.24 38.1 180)
 		(effects
 			(font
-				(size 1 1)
-			)
-			(justify right)
-		)
-	)
-	(hierarchical_label "BMS_OK_SAMPLE"
-		(shape input)
-		(at 142.24 66.04 180)
-		(effects
-			(font
-				(size 1 1)
-			)
-			(justify right)
-		)
-	)
-	(hierarchical_label "12V_COOLANT_SAMPLE"
-		(shape input)
-		(at 105.41 123.19 0)
-		(effects
-			(font
-				(size 1 1)
-			)
-			(justify left)
-		)
-	)
-	(hierarchical_label "12V_BRAKE_LIGHT_SAMPLE"
-		(shape input)
-		(at 105.41 125.73 0)
-		(effects
-			(font
-				(size 1 1)
-			)
-			(justify left)
-		)
-	)
-	(hierarchical_label "DISCHG_SAMPLE"
-		(shape input)
-		(at 142.24 63.5 180)
-		(effects
-			(font
-				(size 1 1)
-			)
-			(justify right)
-		)
-	)
-	(hierarchical_label "IMD_PWM_SAMPLE"
-		(shape input)
-		(at 67.31 156.21 180)
-		(effects
-			(font
-				(size 1 1)
-			)
-			(justify right)
-		)
-	)
-	(hierarchical_label "12V_DTI_SAMPLE"
-		(shape input)
-		(at 105.41 130.81 0)
-		(effects
-			(font
-				(size 1 1)
-			)
-			(justify left)
-		)
-	)
-	(hierarchical_label "SDN_RIGHT_ESTOP_SAMPLE"
-		(shape input)
-		(at 142.24 53.34 180)
-		(effects
-			(font
-				(size 1 1)
-			)
-			(justify right)
-		)
-	)
-	(hierarchical_label "12V_ENERGY_METER_SAMPLE"
-		(shape input)
-		(at 105.41 135.89 0)
-		(effects
-			(font
-				(size 1 1)
-			)
-			(justify left)
-		)
-	)
-	(hierarchical_label "SDN_FRONT_SAMPLE"
-		(shape input)
-		(at 142.24 43.18 180)
-		(effects
-			(font
-				(size 1 1)
-			)
-			(justify right)
-		)
-	)
-	(hierarchical_label "12V_FAN_SAMPLE"
-		(shape input)
-		(at 105.41 118.11 0)
-		(effects
-			(font
-				(size 1 1)
-			)
-			(justify left)
-		)
-	)
-	(hierarchical_label "SDN_HVD_SAMPLE"
-		(shape input)
-		(at 142.24 55.88 180)
-		(effects
-			(font
-				(size 1 1)
-			)
-			(justify right)
-		)
-	)
-	(hierarchical_label "SDN_TSMS_SAMPLE"
-		(shape input)
-		(at 142.24 48.26 180)
-		(effects
-			(font
-				(size 1 1)
-			)
-			(justify right)
-		)
-	)
-	(hierarchical_label "12V_IMD_SAMPLE"
-		(shape input)
-		(at 105.41 115.57 0)
-		(effects
-			(font
-				(size 1 1)
-			)
-			(justify left)
-		)
-	)
-	(hierarchical_label "12V_BMS_SAMPLE"
-		(shape input)
-		(at 105.41 113.03 0)
-		(effects
-			(font
-				(size 1 1)
-			)
-			(justify left)
-		)
-	)
-	(hierarchical_label "IMD_OK_SAMPLE"
-		(shape input)
-		(at 142.24 68.58 180)
-		(effects
-			(font
-				(size 1 1)
-			)
-			(justify right)
-		)
-	)
-	(hierarchical_label "SDN_LATCH_SAMPLE"
-		(shape input)
-		(at 142.24 40.64 180)
-		(effects
-			(font
